Commit message: adds anymal-b urdf from legged-gym

File: urdf/anymal_original.urdf (robot description, URDF)
Before this commit: robot anymal, 21 links, 20 joints
Links:
- added link base_inertia, mass 16.793507758
- link LF_ADAPTER: geometry collision cylinder length=0.32125 radius=0.015; visual mesh filename=package://anymal_b_simple_description/meshes/anymal_foot.dae scale=0.001 0.001 0.001
- link LF_FOOT: mass 0.05 -> None
- link LF_HIP: geometry collision cylinder length=0.03 radius=0.045; collision cylinder length=0.1 radius=0.08
- link LF_SHANK: geometry collision box size=0.08 0.07 0.13; visual mesh filename=package://anymal_b_simple_description/meshes/anymal_shank_l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 scale=0.001 0.001 0.001
- link LF_THIGH: geometry collision box size=0.08 0.04 0.25; collision cylinder length=0.12 radius=0.06
- link LH_ADAPTER: geometry collision cylinder length=0.32125 radius=0.015; visual mesh filename=package://anymal_b_simple_description/meshes/anymal_foot.dae scale=0.001 0.001 0.001
- link LH_FOOT: mass 0.05 -> None
- link LH_HIP: geometry collision cylinder length=0.03 radius=0.045; collision cylinder length=0.1 radius=0.08
- link LH_SHANK: geometry collision box size=0.08 0.07 0.13; visual mesh filename=package://anymal_b_simple_description/meshes/anymal_shank_r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 scale=0.001 0.001 0.001
- link LH_THIGH: geometry collision box size=0.08 0.04 0.25; collision cylinder length=0.12 radius=0.06
- link RF_ADAPTER: geometry collision cylinder length=0.32125 radius=0.015; visual mesh filename=package://anymal_b_simple_description/meshes/anymal_foot.dae scale=0.001 0.001 0.001
- link RF_FOOT: mass 0.05 -> None
- link RF_HIP: geometry collision cylinder length=0.03 radius=0.045; collision cylinder length=0.1 radius=0.08
- link RF_SHANK: geometry collision box size=0.08 0.07 0.13; visual mesh filename=package://anymal_b_simple_description/meshes/anymal_shank_r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 scale=0.001 0.001 0.001
- link RF_THIGH: geometry collision box size=0.08 0.04 0.25; collision cylinder length=0.12 radius=0.06
- link RH_ADAPTER: geometry collision cylinder length=0.32125 radius=0.015; visual mesh filename=package://anymal_b_simple_description/meshes/anymal_foot.dae scale=0.001 0.001 0.001
- link RH_FOOT: mass 0.05 -> None
- link RH_HIP: geometry collision cylinder length=0.03 radius=0.045; collision cylinder length=0.1 radius=0.08
- link RH_SHANK: geometry collision box size=0.08 0.07 0.13; visual mesh filename=package://anymal_b_simple_description/meshes/anymal_shank_l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 scale=0.001 0.001 0.001
- link RH_THIGH: geometry collision box size=0.08 0.04 0.25; collision cylinder length=0.12 radius=0.06
- link base: mass 16.793507758 -> None; geometry collision box size=0.1 0.1 0.07; collision box size=0.1 0.1 0.07
Joints:
- added joint base_to_base_inertia: type fixed, parent base, child base_inertia, origin xyz=0 0 0 rpy=0 0 0
- joint LF_HFE: limit lower=-9.42 upper=9.42 effort=80 velocity=20 -> lower=-9.42 upper=9.42 effort=80 velocity=15.0
- joint LF_KFE: limit lower=-9.42 upper=9.42 effort=80 velocity=20 -> lower=-9.42 upper=9.42 effort=80 velocity=15.0
- joint LH_HFE: limit lower=-9.42 upper=9.42 effort=80 velocity=20 -> lower=-9.42 upper=9.42 effort=80 velocity=15.0
- joint LH_KFE: limit lower=-9.42 upper=9.42 effort=80 velocity=20 -> lower=-9.42 upper=9.42 effort=80 velocity=15.0
- joint RF_HAA: limit lower=-9.42 upper=9.42 effort=80 velocity=20 -> lower=-9.42 upper=9.42 effort=80 velocity=15
- joint RF_HFE: limit lower=-9.42 upper=9.42 effort=80 velocity=20 -> lower=-9.42 upper=9.42 effort=80 velocity=15.0
- joint RF_KFE: limit lower=-9.42 upper=9.42 effort=80 velocity=20 -> lower=-9.42 upper=9.42 effort=80 velocity=15.0
- joint RH_HFE: limit lower=-9.42 upper=9.42 effort=80 velocity=20 -> lower=-9.42 upper=9.42 effort=80 velocity=15.0
- joint RH_KFE: limit lower=-9.42 upper=9.42 effort=80 velocity=20 -> lower=-9.42 upper=9.42 effort=80 velocity=15.0
